File: gate_boost.sch (EAGLE design)
At the start: 57 parts, among them IC1 LM324D, IC2 SP34063A_BOOST_REG

Commit message: prior change to charge pump
Parts:
- C1: value (none) -> 1500pf
- R19: value (none) -> 68k
- R20: value (none) -> 180
- R21: value (none) -> 0.22
- R23: value (none) -> 3k3
- R24: value (none) -> 6k2
Changed lines of the file:
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@@
 <part name="SUPPLY4" library="supply2" deviceset="GND" device=""/>
 <part name="IC2" library="jason_eagle6" deviceset="SP34063A_BOOST_REG" device=""/>
-<part name="R20" library="rcl" deviceset="R-EU_" device="R0805"/>
+<part name="R20" library="rcl" deviceset="R-EU_" device="R0805" value="180"/>
 <part name="SUPPLY5" library="supply2" deviceset="GND" device=""/>
-<part name="C1" library="rcl" deviceset="C-EU" device="C0805"/>
+<part name="C1" library="rcl" deviceset="C-EU" device="C0805" value="1500pf"/>
 <part name="JP1" library="pinhead" deviceset="PINHD-1X3" device=""/>
-<part name="R24" library="rcl" deviceset="R-EU_" device="R0805"/>
-<part name="R23" library="rcl" deviceset="R-EU_" device="R0805"/>
+<part name="R24" library="rcl" deviceset="R-EU_" device="R0805" value="6k2"/>
+<part name="R23" library="rcl" deviceset="R-EU_" device="R0805" value="3k3"/>
 <part name="SUPPLY6" library="supply2" deviceset="V+" device=""/>
-<part name="R21" library="rcl" deviceset="R-EU_" device="R0805"/>
-<part name="R19" library="rcl" deviceset="R-EU_" device="R0805"/>
+<part name="R21" library="rcl" deviceset="R-EU_" device="R0805" value="0.22"/>
+<part name="R19" library="rcl" deviceset="R-EU_" device="R0805" value="68k"/>
 <part name="SUPPLY7" library="supply2" deviceset="GND" device=""/>
 <part name="SUPPLY8" library="supply2" deviceset="GND" device=""/>
@@
 <instance part="SUPPLY4" gate="GND" x="124.46" y="17.78"/>
 <instance part="IC2" gate="G$1" x="243.84" y="81.28"/>
-<instance part="R20" gate="G$1" x="276.86" y="83.82"/>
+<instance part="R20" gate="G$1" x="276.86" y="83.82" smashed="yes">
+<attribute name="NAME" x="273.05" y="85.3186" size="1.778" layer="95"/>
+<attribute name="VALUE" x="274.828" y="82.804" size="1.778" layer="96"/>
+</instance>
 <instance part="SUPPLY5" gate="GND" x="213.36" y="38.1"/>
 <instance part="C1" gate="G$1" x="220.98" y="78.74" rot="R270"/>
@@
 <instance part="R23" gate="G$1" x="236.22" y="43.18" rot="R180"/>
 <instance part="SUPPLY6" gate="1" x="195.58" y="68.58"/>
-<instance part="R21" gate="G$1" x="276.86" y="78.74"/>
+<instance part="R21" gate="G$1" x="276.86" y="78.74" smashed="yes">
+<attribute name="NAME" x="273.05" y="80.2386" size="1.778" layer="95"/>
+<attribute name="VALUE" x="274.32" y="77.978" size="1.778" layer="96"/>
+</instance>
 <instance part="R19" gate="G$1" x="223.52" y="58.42"/>
 <instance part="SUPPLY7" gate="GND" x="269.24" y="38.1"/>

Commit message: charge pump
Parts:
- removed D10, D9: CGRM4001-G, diode:CGRM4001-G
- removed D5, D6, D7, D8: PD3S160, diode:PD3S160
- removed JP1: (no value), pinhead:PINHD-1X3
- removed L1: (no value), wuerth-elektronik:WE-PD_S/M
- removed LED5: (no value), adafruit:LED3MM
- removed PWR1, PWR2: 2.1MMJACKTHM, adafruit:2.1MMJACKTHM
- removed R22: (no value), rcl:R-EU_R0805
- removed R23: 3k3, rcl:R-EU_R0805
- removed R24: 6k2, rcl:R-EU_R0805
- added C10, C11, C12, C5: (no value), resistor:C-EUC0805
- added C6: (no value), rcl:CPOL-EUSMCA
- added C7, C8: 10u, rcl:CPOL-EUSMCA
- added C9: (no value), rcl:CPOL-EUE2-5
- added CLK_LED2: (no value), led:LED3MM
- added IC3: LM27675M5_CHARGEPUMP, jason_eagle6:LM27675M5_CHARGEPUMP
- added IC4: LM358D, linear:LM358D
- added S1: (no value), switch-dil:DIP02YL
- added U$1, U$2: PWR_SOCKET_2_1MM, jason_eagle6:PWR_SOCKET_2_1MM
- C1: value 1500pf -> (none); device rcl:C-EUC0805 -> resistor:C-EUC0805
- C2: device rcl:C-EUC0805 -> resistor:C-EUC0805
- C3, C4: device rcl:CPOL-EUE2.5-6 -> resistor:C-EUC0805
- D1, D2, D3, D4: value PD3S160 -> MBR0520LT; device diode:PD3S160 -> diode:MBR0520LT
- IC1: value LM324D -> LM358D; device linear:LM324D -> linear:LM358D
- IC2: value SP34063A_BOOST_REG -> REG1117; device jason_eagle6:SP34063A_BOOST_REG -> burr-brown:REG1117
- IN1, IN2, IN3, IN4, OUT1, OUT2, OUT3, OUT4: value TRUCONNECTJACK -> VERTICAL_3_5MM_SOCKET; device jason_eagle6:TRUCONNECTJACK -> jason_eagle6:VERTICAL_3_5MM_SOCKET
- LED1, LED2, LED3, LED4: device adafruit:LED3MM -> led:LED3MM
- R1, R10, R13, R2: value (none) -> 1K
- R12, R16, R17, R18, R6, R9: value (none) -> 100k
- R19: value 68k -> (none)
- R20: value 180 -> (none)
- R21: value 0.22 -> 1K
Connections:
- removed net N$18: IC1C.OUT, LED3.A, R14.1
- removed net N$22: IC2.DR_C, R20.1
- removed net N$24: C4.+, D10.C, IC2.VCC, R21.1
- removed net N$25: D10.A, PWR1.RING, PWR2.RING
- removed net N$27: LED1.C, R9.2
- removed net N$30: LED2.C, R11.2
- removed net N$31: LED3.C, R13.2
- removed net N$32: LED4.C, R15.2
- removed net N$34: LED5.C, R22.2
- removed net N$6: D5.C, D6.A, IC1C.+IN, R5.2, R6.2
- removed net V+: C2.2, C3.+, D2.C, D4.C, D6.C, D8.C, D9.C, IC1P.V+, LED5.A, R18.2, R19.1
- new net +10V: C6.+, D1.C, D3.A, D4.A, IC3.OUT
- new net +5V: C12.1, C7.+, CLK_LED2.A, D1.A, IC2.VOUT, IC3.V+, R16.2, R6.2
- new net IN1: IN1.4, LED1.A, R12.2
- new net IN2: IN2.4, LED2.A, R9.2
- new net IN3: IN3.4, LED3.A, R17.2
- new net IN4: IN4.4, LED4.A, R18.2
- new net N$38: C8.+, IC3.CAP+
- new net N$39: C8.-, IC3.CAP-
- new net VGATE1: C10.1, D3.C, IC4P.V+, S1.1
- new net VGATE2: C3.1, D4.C, IC1P.V+, S1.2
- new net VIN: C11.1, C9.+, D2.C, IC2.VIN, S1.3, S1.4
- net GND: now also C10.2, C11.2, C12.2, C2.2, C3.2, C4.2, C5.2, C6.-, C7.-, C9.-, IC3.GND, IC3.SD, IC4P.V-, IN1.2, IN2.2, IN3.2, IN4.2, OUT1.2, OUT2.2, OUT3.2, OUT4.2, R1.2, R10.2, R13.2, R2.2, R21.2, U$1.PIN, U$2.PIN; no longer C2.1, C3.-, C4.-, D1.A, D3.A, D5.A, D7.A, IC2.SW_E, IN1.SLEEVE, IN2.SLEEVE, IN3.SLEEVE, IN4.SLEEVE, OUT1.SLEEVE, OUT2.SLEEVE, OUT3.SLEEVE, OUT4.SLEEVE, PWR1.TIP, PWR2.TIP, R1.1, R11.1, R13.1, R17.1, R22.1, R24.1, R3.1, R5.1, R9.1
- net N$1: now also IC4A.-IN, IC4B.-IN, R6.1, R7.2; no longer IN1.TIP, IN1.TIP_NC, R2.1
- net N$10: now also IC1B.OUT, R14.1, R19.1; no longer IC1A.-IN, IC1B.-IN, IC1C.-IN, IC1D.-IN, R17.2, R18.1
- net N$11: now also IC1A.OUT, R20.1, R3.1; no longer OUT1.TIP, OUT1.TIP_NC, R10.2
- net N$12: now also IC4B.OUT, R4.1, R8.1; no longer OUT2.TIP, OUT2.TIP_NC, R12.2
- net N$13: now also IC1A.-IN, IC1B.-IN, R15.2, R16.1; no longer OUT3.TIP, OUT3.TIP_NC, R14.2
- net N$14: now also LED3.C, R2.1; no longer OUT4.TIP, OUT4.TIP_NC, R16.2
- net N$15: now also LED4.C, R1.1; no longer C1.1, IC2.TC
- net N$16: now also IC1A.+IN, R17.1, R20.2; no longer D9.A, IC2.SW_C, L1.1
- net N$17: now also IC1B.+IN, R18.1, R19.2; no longer IC1B.OUT, LED2.A, R12.1
- net N$19: now also C5.1, OUT1.4, R5.2; no longer IC1D.OUT, LED4.A, R16.1
- net N$2: now also LED1.C, R13.1; no longer IN2.TIP, IN2.TIP_NC, R4.1
- net N$20: now also C4.1, OUT2.4, R4.2; no longer IC2.COMP, JP1.2, R19.2, R23.1
- net N$21: now also D2.A, U$1.BARREL, U$2.BARREL; no longer JP1.1, R23.2, R24.2
- net N$23: now also CLK_LED2.C, R21.1; no longer IC2.SENS, L1.2, R20.2, R21.2
- net N$3: now also LED2.C, R10.1; no longer IN3.TIP, IN3.TIP_NC, R6.1
- net N$4: now also IC4A.+IN, R11.2, R12.1; no longer IN4.TIP, IN4.TIP_NC, R8.1
- net N$5: now also IC4B.+IN, R9.1; no longer D7.C, D8.A, IC1D.+IN, R7.2
- net N$7: now also C1.1, OUT3.4; no longer D3.C, D4.A, IC1B.+IN, R4.2
- net N$8: now also C2.1, OUT4.4, R14.2; no longer D1.C, D2.A, IC1A.+IN, R1.2, R2.2
- net N$9: now also IC4A.OUT, R11.1, R5.1; no longer IC1A.OUT, LED1.A, R10.1
Other:
- note added: "10V CHARGE PUMP"
- note added: "CC-BY-SA"
- note added: "CVOCD GATE BOOST"
- note added: "Sixty four pixels limited"
- note added: "VERSION 1 - 10jan19"
- moved on the sheet: C1, C2, IC1A, IC1B, LED1, LED2, LED3, LED4, R1, R10, R11, R12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

Commit message: getting there
Parts:
- C10, C11: value (none) -> 10u; device resistor:C-EUC0805 -> rcl:CPOL-EUSMCA
- C12: device resistor:C-EUC0805 -> rcl:CPOL-EUE2-5
- C6: device rcl:CPOL-EUSMCA -> resistor:C-EUC0805
- C7, C8: value 10u -> (none); device rcl:CPOL-EUSMCA -> resistor:C-EUC0805
- C9: device rcl:CPOL-EUE2-5 -> rcl:CPOL-EUSMCA
- IC2: value REG1117 -> LM358D; device burr-brown:REG1117 -> linear:LM358D
- IC4: value LM358D -> REG1117; device linear:LM358D -> burr-brown:REG1117
- R10, R13, R21: value 1K -> (none)
- R17: value 100k -> 1K
- R18, R9: value 100k -> (none)
- R2: value 1K -> 100k
- R3, R5, R7: value (none) -> 1K
- R4, R8: value (none) -> 100k
- renumbered CLK_LED2 to PWR, LED1 to A, LED2 to B, LED3 to C, LED4 to D, S1 to SW1
Connections:
- net +10V: now also C9.+; no longer C6.+
- net +5V: now also C10.+, C8.1, IC4.VOUT, R12.2; no longer C12.1, C7.+, IC2.VOUT, R6.2
- net GND: now also C10.-, C12.-, C6.2, C7.2, C8.2, IC2P.V-, IC4.GND, R11.1, R17.2, R3.2, R5.2, R7.2; no longer C10.2, C11.2, C12.2, C6.-, C7.-, IC2.GND, IC4P.V-, R10.2, R13.2, R2.2, R21.2, R7.1
- net IN1: now also R2.2; no longer R12.2
- net IN2: now also R4.2; no longer R9.2
- net IN3: now also R6.2; no longer R17.2
- net IN4: now also R8.2; no longer R18.2
- net N$1: now also IC1A.-IN, IC1B.-IN, R11.2, R12.1; no longer IC4A.-IN, IC4B.-IN, R6.1, R7.2
- net N$10: now also IC2B.OUT, R21.1; no longer IC1B.OUT, R19.1
- net N$11: now also IC2A.OUT, R13.1; no longer IC1A.OUT, R3.1
- net N$12: now also IC1B.OUT, R10.1, R19.1; no longer IC4B.OUT, R4.1, R8.1
- net N$13: now also IC2A.-IN, IC2B.-IN; no longer IC1A.-IN, IC1B.-IN
- net N$14: now also R5.1; no longer R2.1
- net N$15: now also R7.1; no longer R1.1
- net N$16: now also IC2A.+IN, R13.2, R6.1; no longer IC1A.+IN, R17.1, R20.2
- net N$17: now also IC2B.+IN, R14.2, R8.1; no longer IC1B.+IN, R18.1, R19.2
- net N$19: now also C3.1, R18.2; no longer C5.1, R5.2
- net N$2: now also R1.1; no longer R13.1
- net N$20: now also R19.2; no longer R4.2
- net N$23: now also R17.1; no longer R21.1
- net N$3: now also R3.1; no longer R10.1
- net N$38: now also C11.+; no longer C8.+
- net N$39: now also C11.-; no longer C8.-
- net N$4: now also IC1A.+IN, R2.1, R9.2; no longer IC4A.+IN, R11.2, R12.1
- net N$5: now also IC1B.+IN, R10.2, R4.1; no longer IC4B.+IN, R8.2, R9.1
- net N$7: now also C5.1, R20.2; no longer C1.1, R3.2
- net N$8: now also C6.1, R21.2; no longer C2.1, R14.2
- net N$9: now also IC1A.OUT, R18.1, R9.1; no longer IC4A.OUT, R11.1, R5.1
- net VGATE1: now also C1.1, IC1P.V+; no longer C10.1, IC4P.V+
- net VGATE2: now also C2.1, IC2P.V+; no longer C3.1, IC1P.V+
- net VIN: now also C12.+, C7.1, IC4.VIN; no longer C11.1, C9.+, IC2.VIN
Other:
- moved on the sheet: C1, C2, C3, C5, C9, IC1A, IC1B, R1, R10, R11, R12, R13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

Commit message: component values
Parts:
- R13, R14: value (none) -> 2m2
- R15: value (none) -> 47k
- R16: value 100k -> 47k
- R20, R21: value (none) -> 1k
Changed lines of the file:
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@@
 <part name="C5" library="resistor" deviceset="C-EU" device="C0805"/>
 <part name="C6" library="resistor" deviceset="C-EU" device="C0805"/>
-<part name="R20" library="rcl" deviceset="R-EU_" device="R0805"/>
+<part name="R20" library="rcl" deviceset="R-EU_" device="R0805" value="1k"/>
 <part name="GND2" library="SparkFun" deviceset="GND" device=""/>
-<part name="R21" library="rcl" deviceset="R-EU_" device="R0805"/>
+<part name="R21" library="rcl" deviceset="R-EU_" device="R0805" value="1k"/>
 <part name="IC2" library="linear" deviceset="LM358" device="D"/>
-<part name="R15" library="rcl" deviceset="R-EU_" device="R0805"/>
-<part name="R16" library="rcl" deviceset="R-EU_" device="R0805" value="100k"/>
+<part name="R15" library="rcl" deviceset="R-EU_" device="R0805" value="47k"/>
+<part name="R16" library="rcl" deviceset="R-EU_" device="R0805" value="47k"/>
 <part name="GND3" library="SparkFun" deviceset="GND" device=""/>
 <part name="SUPPLY1" library="supply2" deviceset="+5V" device=""/>
@@
 <part name="R6" library="rcl" deviceset="R-EU_" device="R0805" value="100k"/>
 <part name="R8" library="rcl" deviceset="R-EU_" device="R0805" value="100k"/>
-<part name="R14" library="rcl" deviceset="R-EU_" device="R0805"/>
-<part name="R13" library="rcl" deviceset="R-EU_" device="R0805"/>
+<part name="R14" library="rcl" deviceset="R-EU_" device="R0805" value="2m2"/>
+<part name="R13" library="rcl" deviceset="R-EU_" device="R0805" value="2m2"/>
 <part name="C2" library="resistor" deviceset="C-EU" device="C0805"/>
 <part name="OUT1" library="jason_eagle6" deviceset="VERTICAL_3_5MM_SOCKET" device=""/>

Commit message: aye
Parts:
- R10, R9: value (none) -> 2m2
- R11: value (none) -> 47k
- R12: value 100k -> 47k
- R18, R19: value (none) -> 1k
Changed lines of the file:
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@@
 <part name="C3" library="resistor" deviceset="C-EU" device="C0805"/>
 <part name="C4" library="resistor" deviceset="C-EU" device="C0805"/>
-<part name="R18" library="rcl" deviceset="R-EU_" device="R0805"/>
+<part name="R18" library="rcl" deviceset="R-EU_" device="R0805" value="1k"/>
 <part name="GND16" library="SparkFun" deviceset="GND" device=""/>
-<part name="R19" library="rcl" deviceset="R-EU_" device="R0805"/>
+<part name="R19" library="rcl" deviceset="R-EU_" device="R0805" value="1k"/>
 <part name="IC3" library="jason_eagle6" deviceset="LM27675M5_CHARGEPUMP" device=""/>
 <part name="D1" library="diode" deviceset="MBR0520LT" device=""/>
@@
 <part name="SUPPLY7" library="supply2" deviceset="+10V" device=""/>
 <part name="IC1" library="linear" deviceset="LM358" device="D"/>
-<part name="R11" library="rcl" deviceset="R-EU_" device="R0805"/>
-<part name="R12" library="rcl" deviceset="R-EU_" device="R0805" value="100k"/>
+<part name="R11" library="rcl" deviceset="R-EU_" device="R0805" value="47k"/>
+<part name="R12" library="rcl" deviceset="R-EU_" device="R0805" value="47k"/>
 <part name="GND11" library="SparkFun" deviceset="GND" device=""/>
 <part name="SUPPLY2" library="supply2" deviceset="+5V" device=""/>
@@
 <part name="R2" library="rcl" deviceset="R-EU_" device="R0805" value="100k"/>
 <part name="R4" library="rcl" deviceset="R-EU_" device="R0805" value="100k"/>
-<part name="R10" library="rcl" deviceset="R-EU_" device="R0805"/>
-<part name="R9" library="rcl" deviceset="R-EU_" device="R0805"/>
+<part name="R10" library="rcl" deviceset="R-EU_" device="R0805" value="2m2"/>
+<part name="R9" library="rcl" deviceset="R-EU_" device="R0805" value="2m2"/>
 <part name="C1" library="resistor" deviceset="C-EU" device="C0805"/>
 <part name="C" library="led" deviceset="LED" device="3MM"/>

Commit message: V2 additional schottky on VIN
Parts:
- added D5: MBR0520LT, diode:MBR0520LT
Connections:
- new net N$6: D3.C, SW1.3, SW1.4
- net +10V: now also D5.A; no longer D3.A
- net VGATE1: now also D4.C; no longer D3.C
- net VGATE2: now also D5.C; no longer D4.C
- net VIN: now also D3.A; no longer SW1.3, SW1.4
Other:
- note added: "5V REGULATOR"
- note added: "GATE VOLTAGE SELECTION"
- note added: "OUTPUT BUFFERS 1/2"
- note added: "OUTPUT BUFFERS 3/4"
- note added: "VERSION 2 - 13feb19"
- note removed: "VERSION 1 - 10jan19"
- moved on the sheet: D3, D4
Changed lines of the file:
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@@
 <part name="GND15" library="SparkFun" deviceset="GND" device=""/>
 <part name="GND23" library="SparkFun" deviceset="GND" device=""/>
-<part name="D3" library="diode" deviceset="MBR0520LT" device=""/>
 <part name="D4" library="diode" deviceset="MBR0520LT" device=""/>
+<part name="D5" library="diode" deviceset="MBR0520LT" device=""/>
 <part name="U$4" library="microbuilder" deviceset="VIN" device=""/>
 <part name="GND24" library="SparkFun" deviceset="GND" device=""/>
+<part name="D3" library="diode" deviceset="MBR0520LT" device=""/>
 </parts>
 <sheets>
@@
 <text x="49.276" y="0.254" size="3.81" layer="91">10V CHARGE PUMP</text>
 <text x="2.286" y="-31.75" size="5.08" layer="91">CVOCD GATE BOOST</text>
-<text x="2.54" y="-38.1" size="5.08" layer="91">VERSION 1 - 10jan19</text>
+<text x="2.54" y="-38.1" size="5.08" layer="91">VERSION 2 - 13feb19</text>
 <text x="2.54" y="-45.72" size="3.81" layer="91">Sixty four pixels limited</text>
 <text x="2.54" y="-50.8" size="3.81" layer="91">CC-BY-SA</text>
+<text x="-6.604" y="45.974" size="3.81" layer="91">5V REGULATOR</text>
+<text x="67.056" y="68.834" size="3.81" layer="91">GATE VOLTAGE
+SELECTION</text>
+<text x="204.216" y="40.894" size="3.81" layer="91">OUTPUT
+BUFFERS 1/2</text>
+<text x="206.756" y="-50.546" size="3.81" layer="91">OUTPUT
+BUFFERS 3/4</text>
 </plain>
 <instances>
@@
 <instance part="GND15" gate="1" x="162.56" y="33.02"/>
 <instance part="GND23" gate="1" x="162.56" y="-58.42"/>
-<instance part="D3" gate="G$1" x="111.76" y="40.64" rot="R90"/>
-<instance part="D4" gate="G$1" x="114.3" y="45.72" rot="R90"/>
-<instance part="U$4" gate="G$1" x="111.76" y="88.9"/>
+<instance part="D4" gate="G$1" x="111.76" y="40.64" rot="R90"/>
+<instance part="D5" gate="G$1" x="114.3" y="45.72" rot="R90"/>
+<instance part="U$4" gate="G$1" x="111.76" y="101.6"/>
 <instance part="GND24" gate="1" x="-27.94" y="15.24"/>
+<instance part="D3" gate="G$1" x="111.76" y="93.98" rot="R270"/>
 </instances>
 <busses>
@@
 <pinref part="SUPPLY7" gate="G$1" pin="+10V"/>
 <wire x1="96.52" y1="40.64" x2="96.52" y2="35.56" width="0.1524" layer="91"/>
-<pinref part="D3" gate="G$1" pin="A"/>
+<pinref part="D4" gate="G$1" pin="A"/>
 <wire x1="96.52" y1="35.56" x2="111.76" y2="35.56" width="0.1524" layer="91"/>
 <wire x1="111.76" y1="35.56" x2="111.76" y2="38.1" width="0.1524" layer="91"/>
-<pinref part="D4" gate="G$1" pin="A"/>
+<pinref part="D5" gate="G$1" pin="A"/>
 <wire x1="111.76" y1="35.56" x2="114.3" y2="35.56" width="0.1524" layer="91"/>
 <wire x1="114.3" y1="35.56" x2="114.3" y2="43.18" width="0.1524" layer="91"/>
@@
 </segment>
 <segment>
-<pinref part="D4" gate="G$1" pin="C"/>
+<pinref part="D5" gate="G$1" pin="C"/>
 <pinref part="SW1" gate="1" pin="2"/>
 <wire x1="114.3" y1="48.26" x2="114.3" y2="60.96" width="0.1524" layer="91"/>
@@
 </segment>
 <segment>
-<pinref part="SW1" gate="1" pin="4"/>
-<wire x1="111.76" y1="81.28" x2="111.76" y2="86.36" width="0.1524" layer="91"/>
-<wire x1="111.76" y1="86.36" x2="114.3" y2="86.36" width="0.1524" layer="91"/>
-<pinref part="SW1" gate="1" pin="3"/>
-<wire x1="114.3" y1="86.36" x2="114.3" y2="81.28" width="0.1524" layer="91"/>
+<pinref part="D3" gate="G$1" pin="A"/>
 <pinref part="U$4" gate="G$1" pin="VIN"/>
-<wire x1="111.76" y1="88.9" x2="111.76" y2="86.36" width="0.1524" layer="91"/>
-<junction x="111.76" y="86.36"/>
+<wire x1="111.76" y1="96.52" x2="111.76" y2="101.6" width="0.1524" layer="91"/>
 </segment>
 </net>
@@
 </segment>
 <segment>
-<pinref part="D3" gate="G$1" pin="C"/>
+<pinref part="D4" gate="G$1" pin="C"/>
 <pinref part="SW1" gate="1" pin="1"/>
 <wire x1="111.76" y1="43.18" x2="111.76" y2="63.5" width="0.1524" layer="91"/>
@@
 </segment>
 </net>
+<net name="N$6" class="0">
+<segment>
+<pinref part="SW1" gate="1" pin="4"/>
+<wire x1="111.76" y1="81.28" x2="111.76" y2="86.36" width="0.1524" layer="91"/>
+<wire x1="111.76" y1="86.36" x2="114.3" y2="86.36" width="0.1524" layer="91"/>
+<pinref part="SW1" gate="1" pin="3"/>
+<wire x1="114.3" y1="86.36" x2="114.3" y2="81.28" width="0.1524" layer="91"/>
+<pinref part="D3" gate="G$1" pin="C"/>
+<wire x1="111.76" y1="91.44" x2="111.76" y2="86.36" width="0.1524" layer="91"/>
+<junction x="111.76" y="86.36"/>
+</segment>
+</net>
 </nets>
 </sheet>
@@
 </schematic>
 </drawing>
+<compatibility>
+<note version="6.3" minversion="6.2.2" severity="warning">
+Since Version 6.2.2 text objects can contain more than one line,
+which will not be processed correctly with this version.
+</note>
+</compatibility>
 </eagle>
